File: watter.flow.metter/pcb/watter.flow.metter.brd (EAGLE design)
At the start: 131.9 x 48.2 mm, 25 parts, among them Q1 BC546A

Commit message: add timer for periodical switching relay
Parts:
- removed DISPLAY: OLED_0.96_I2C, tft_1.8_1.44_oled_0.96:OLED_0.96_I2C
- added U$1: DISPLAY-OLED-128X64-I2C, diy-modules:DISPLAY-OLED-128X64-I2C
Connections:
- net 3.3V: now also U$1.2; no longer DISPLAY.VCC
- net GND: now also U$1.1; no longer DISPLAY.GND
- net SCL: now also U$1.3; no longer DISPLAY.SCL
- net SDA: now also U$1.4; no longer DISPLAY.SDA
Routing:
- net 3.3V: track 51.8 -> 49.2 mm
Changed lines of the file:
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@@
 <elements>
 <element name="U$5" library="Arduino" package="NANO" value="NANO" x="106.045" y="14.2875" smashed="yes"/>
-<element name="DISPLAY" library="tft_1.8_1.44_oled_0.96" package="OLED_0.96_I2C" value="OLED_0.96_I2C" x="56.1975" y="30.7975"/>
 <element name="RELE1" library="relay" library_urn="urn:adsk.eagle:library:339" package="JS-M" value="JS-M1-9V-4" x="22.86" y="9.2075" smashed="yes">
 <attribute name="MF" value="" x="22.86" y="9.2075" size="1.778" layer="27" display="off"/>
@@
 <attribute name="VALUE" x="52.6669" y="11.7475" size="1.27" layer="27" ratio="10"/>
 </element>
+<element name="U$1" library="diy-modules" package="DISPLAY-OLED-128X64-I2C" value="DISPLAY-OLED-128X64-I2C" x="55.88" y="29.845"/>
 </elements>
 <signals>
 <signal name="GND">
-<contactref element="DISPLAY" pad="GND"/>
 <contactref element="U$6" pad="GND@1"/>
 <contactref element="U$2" pad="P$5"/>
@@
 <wire x1="52.54625" y1="6.35" x2="52.54625" y2="7.77875" width="0.8128" layer="16"/>
 <contactref element="U$6" pad="GND@2"/>
-<wire x1="54.61" y1="42.385" x2="54.5675" y2="42.4275" width="0.8128" layer="16"/>
 <polygon width="0.8128" layer="16" isolate="0.6096">
 <vertex x="34.44875" y="48.10125"/>
@@
 <wire x1="23.97125" y1="12.85875" x2="34.925" y2="12.85875" width="0.8128" layer="16"/>
 <wire x1="34.925" y1="12.85875" x2="34.925" y2="12.3825" width="0.8128" layer="16"/>
+<contactref element="U$1" pad="1"/>
+<wire x1="78.105" y1="42.2275" x2="52.07" y2="42.545" width="0" layer="19" extent="1-1"/>
 </signal>
 <signal name="VCC">
@@
 <signal name="SDA">
 <contactref element="U$5" pad="A4"/>
-<contactref element="DISPLAY" pad="SDA"/>
 <contactref element="U$6" pad="SDA@2"/>
 <wire x1="83.185" y1="44.45" x2="59.69" y2="44.45" width="0.4064" layer="16"/>
@@
 <wire x1="88.265" y1="40.16375" x2="83.185" y2="40.16375" width="0.4064" layer="16"/>
 <wire x1="59.69" y1="44.45" x2="59.69" y2="42.4275" width="0.4064" layer="16"/>
-<wire x1="59.69" y1="42.4275" x2="59.6475" y2="42.4275" width="0.4064" layer="16"/>
+<contactref element="U$1" pad="4"/>
+<wire x1="59.69" y1="42.545" x2="59.69" y2="42.4275" width="0" layer="19" extent="16-16"/>
 </signal>
 <signal name="SCL">
 <contactref element="U$5" pad="A5"/>
-<contactref element="DISPLAY" pad="SCL"/>
 <contactref element="U$6" pad="SCL@2"/>
 <wire x1="85.80565625" y1="45.56125" x2="99.695" y2="45.56125" width="0.4064" layer="16"/>
@@
 <wire x1="85.725" y1="45.48059375" x2="85.80565625" y2="45.56125" width="0.4064" layer="16"/>
 <wire x1="57.15" y1="45.56125" x2="57.15" y2="42.4275" width="0.4064" layer="16"/>
-<wire x1="57.15" y1="42.4275" x2="57.1075" y2="42.4275" width="0.4064" layer="16"/>
+<contactref element="U$1" pad="3"/>
+<wire x1="57.15" y1="42.545" x2="57.15" y2="42.4275" width="0" layer="19" extent="16-16"/>
 </signal>
 <signal name="N$41">
@@
 <contactref element="U$5" pad="3.3V"/>
 <contactref element="U$6" pad="VCC@2"/>
-<wire x1="80.645" y1="38.4703875" x2="80.645" y2="42.2275" width="0.508" layer="16"/>
-<wire x1="80.645" y1="38.4703875" x2="80.645" y2="38.4175" width="0.508" layer="16"/>
+<wire x1="80.645" y1="38.4175" x2="80.645" y2="42.2275" width="0.508" layer="16"/>
 <wire x1="80.645" y1="38.4175" x2="95.885" y2="38.4175" width="0.508" layer="16"/>
-<contactref element="DISPLAY" pad="VCC"/>
-<wire x1="52.07" y1="42.385" x2="52.0275" y2="42.4275" width="0.8128" layer="16"/>
-<wire x1="52.0275" y1="42.4275" x2="52.07" y2="42.4275" width="0.508" layer="16"/>
-<wire x1="52.07" y1="42.4275" x2="52.07" y2="38.4175" width="0.508" layer="16"/>
-<wire x1="52.07" y1="38.4175" x2="80.645" y2="38.4175" width="0.508" layer="16"/>
-<wire x1="80.645" y1="38.4175" x2="80.645" y2="38.4703875" width="0.508" layer="16"/>
+<wire x1="80.645" y1="38.4175" x2="54.61" y2="38.4175" width="0.508" layer="16"/>
+<contactref element="U$1" pad="2"/>
+<wire x1="54.61" y1="38.4175" x2="54.61" y2="42.545" width="0.508" layer="16"/>
 </signal>
 </signals>
