File: watter.flow.metter/pcb/watter.flow.metter.2.brd (EAGLE design)
At the start: 98.1 x 99.9 mm, 35 parts, among them J1 22-05-7028-02, Q1 BC546A

Commit message: add scoretable
Parts:
- removed ARDUINO_NANO1: ARDUINO-NANO-3.0, diy-modules:ARDUINO-NANO-3.0
- removed B1, B2, B3: (no value), switch-omron:B3F-10XX
- removed DS3231: RTC-DS3231-AT24C32, diy-modules:RTC-DS3231-AT24C32
- removed J1: 22-05-7028-02, con-molex:7395-02
- removed JP1: (no value), pinhead:1X02
- removed JP2: (no value), pinhead:1X03
- removed R6, R7, R8, R9: (no value), rcl:M1206
Connections:
- removed net 3.3V1: ARDUINO_NANO1.J2.13, ARDUINO_NANO1.J2.14, DS3231.J2.3, R9.2
- removed net D61: ARDUINO_NANO1.J1.7, JP2.2
- removed net GND2: ARDUINO_NANO1.J1.4, ARDUINO_NANO1.J2.2, B1.3, B2.3, B3.3, DS3231.J2.4, J1.2, JP1.1, JP2.3
- removed net N$11: ARDUINO_NANO1.J1.11, B1.1, R6.1
- removed net N$12: ARDUINO_NANO1.J1.12, B2.1, R7.1
- removed net N$13: ARDUINO_NANO1.J1.13, B3.1, R8.1
- removed net N$14: DS3231.J1.6
- removed net N$15: DS3231.J1.5
- removed net N$16: ARDUINO_NANO1.J2.1
- removed net N$34: ARDUINO_NANO1.J2.11, JP1.2, R9.1
- removed net SCL1: ARDUINO_NANO1.J2.7, DS3231.J2.1
- removed net SDA1: ARDUINO_NANO1.J2.8, DS3231.J2.2
- removed net VCC2: ARDUINO_NANO1.J2.4, J1.1, JP2.1, R6.2, R7.2, R8.2
Routing:
- net N$13: track 104.4 -> 0.00 mm
- net N$12: track 90.8 -> 0.00 mm, vias 2 -> 0
- net N$11: track 86.7 -> 0.00 mm, vias 1 -> 0
- net 3.3V1: track 47.9 -> 0.00 mm
- net VCC2: track 39.0 -> 0.00 mm, vias 1 -> 0
- net N$34: track 35.4 -> 0.00 mm
- net SDA1: track 28.4 -> 0.00 mm
- net SCL1: track 25.7 -> 0.00 mm
- net SCL: track 71.2 -> 56.0 mm
- net GND: track 39.3 -> 53.0 mm
- net D61: track 13.2 -> 0.00 mm
- net N$21: track 5.40 -> 0.00 mm
- net N$18: track 5.24 -> 0.00 mm
- net N$17: track 5.08 -> 0.00 mm
- net SDA: track 67.7 -> 62.9 mm
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- removed copper zone on layer 16, net GND2
- removed copper zone on layer 1, net VCC2
Other:
- board size 98.1 x 99.9 mm -> 98.1 x 71 mm
- board text removed: "NEO MATRIX CLOCK"

Commit message: add terminal
Parts:
- removed Q1: BC546A, transistor-npn:TO92-EBC
- added Q4: 2N2222, transistor-npn:TO92
- R1, R2, R3: value (none) -> 10k
- R4: value (none) -> 330
- R5: value (none) -> 5k6
Connections:
- net GND: now also Q4.3; no longer Q1.E
- net N$41: now also Q4.1; no longer Q1.C
- net N$7: now also Q4.2; no longer Q1.B
Routing:
- net N$41: track 36.8 -> 38.2 mm
- net N$7: track 8.61 -> 7.51 mm
